Commit message: last update

File: urdf/anymal_rviz.urdf (robot description, URDF)
Before this commit: robot anymal, 77 links, 76 joints
Links:
- added link rot_y
- added link rot_z
- added link trans_x
- added link trans_y
- added link trans_z
- added link world
Joints:
- added joint rot_x: type continuous, parent rot_y, child base, axis 1 0 0
- added joint rot_y: type continuous, parent rot_z, child rot_y, axis 0 1 0
- added joint rot_z: type continuous, parent trans_z, child rot_z, axis 0 0 1
- added joint trans_x: type prismatic, parent world, child trans_x, axis 1 0 0, limit lower=-50 upper=50 effort=80 velocity=7.5
- added joint trans_y: type prismatic, parent trans_x, child trans_y, axis 0 1 0, limit lower=-50 upper=50 effort=80 velocity=7.5
- added joint trans_z: type prismatic, parent trans_y, child trans_z, axis 0 0 1, limit lower=-50 upper=50 effort=80 velocity=7.5
